Commit message: poprawa do ziemi( trzecie ramie)

File: lab_two/urdf/dynamic.urdf (robot description, URDF)
Before this commit: robot robot, 5 links, 4 joints
Joints:
- joint ARM2_ARM3: limit lower=${BASE_height/-2} upper=${BASE_height/2} effort=1000.0 velocity=0.5 -> lower=${BASE_height/-2} upper=${ARM3_upper_limit} effort=1000.0 velocity=0.5
