Commit message: zad 1 lab 3

File: lab_3/urdf/dynamic.urdf (robot description, URDF)
Before this commit: robot robot, 5 links, 4 joints
Joints:
- joint ARM1_ARM2: axis (none) -> 0 0 1; type fixed -> continuous
- joint ARM2_ARM3: axis (none) -> 0 0 1; limit (none) -> lower=${BASE_height/-2} upper=${ARM3_upper_limit} effort=1000.0 velocity=0.5; type fixed -> prismatic
- joint BASE_ARM1: axis (none) -> 0 0 1; type fixed -> continuous
